File: Adafruit Qualia Driver.brd (EAGLE design)
At the start: 45 x 85 mm, 62 parts, among them IC1 ATTINY85-20S, Q1 DMN10H170SK3-13, T1 IRLML2246, U1 LT3754, U2 MCP16321T-330E/NG, X1 0472720001, X2 FH35-51S-0.3SHW(50), X3 2.1mm

Commit message: right version
Parts:
- added R6: 20K, microbuilder:_0805MP
- added T2: IRLML2246, zetex:SOT-23
- D1: value B260A-13-F -> PDS560-13; device microbuilder:SMADIODE -> microbuilder:POWERDI-5
- Q1: value DMN10H170SK3-13 -> IRLR024NTRPBF
- SW1, SW2, SW3: value (none) -> SPST_TACT-EVQQ2; device microbuilder:BTN_CK_KSS -> adafruit:EVQ-Q2
- X2: value FH35-51S-0.3SHW(50) -> 502250-5191
- moved SW1 73.4 mm to (14.0, 73.7), turned to 90 degrees
- moved SW2 70.9 mm to (5.33, 73.7), turned to 270 degrees
- moved SW3 70.9 mm to (27.9, 73.7), turned to 90 degrees
- moved IC1 63.0 mm to (39.6, 75.8)
- moved D2 56.6 mm to (34.9, 69.3), turned to 270 degrees
- moved ISP1 56.5 mm to (40.0, 69.5), turned to 90 degrees
- moved JP1 55.4 mm to (21.8, 67.1)
- moved R14 54.6 mm to (25.1, 67.1), turned to 180 degrees
- moved L2 11.0 mm to (38.3, 38.0)
- moved SJ1 10.8 mm to (39.0, 33.8)
- moved D1 10.0 mm to (21.5, 57.5), turned to 270 degrees
- moved C1 10.0 mm to (4.00, 41.0)
- moved C10 10.0 mm to (43.4, 50.5)
- moved C11 10.0 mm to (30.4, 46.6)
- moved C12 10.0 mm to (41.7, 45.0)
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Connections:
- removed net N$18: ON/OFF.P2, R7.1, T1.3
- new net DPP: R6.2, T2.2, X1.20
- new net ON/OFF: ON/OFF.P2, R6.1, R7.1, T1.3, T2.3
- net 3.3V: now also T2.1; no longer X1.20
- net BDOWN: now also SW2.B, SW2.B'; no longer SW3.P$2
- net BUP: now also SW1.B, SW1.B'; no longer SW2.P$2
- net GND: now also SW1.A, SW1.A', SW2.A, SW2.A', SW3.A; no longer SW1.P$1, SW2.P$1, SW3.P$1
- net MOSI: now also SW3.B; no longer SW1.P$2
- net N$25: now also D1.A1, D1.A2; no longer D1.A
Routing:
- net ON/OFF: track 0.00 -> 96.5 mm, vias 0 -> 2
- net VCC: track 94.7 -> 183.4 mm, vias 6 -> 8
- net BDOWN: track 17.2 -> 51.4 mm
- net N$18: track 31.8 -> 0.00 mm
- net DPP: track 0.00 -> 18.1 mm
- net N$21: track 18.7 -> 2.59 mm
- net PWM: track 67.6 -> 51.9 mm
- net GND: track 49.0 -> 60.9 mm, vias 36 -> 40
- net N$27: track 7.23 -> 18.2 mm
- net RST: track 8.22 -> 14.7 mm, vias 0 -> 1
- net BUP: track 28.9 -> 34.6 mm
- net 3.3V: track 27.9 -> 31.0 mm
- net MOSI: track 19.4 -> 20.8 mm
- net SCLK: track 14.2 -> 13.1 mm, vias 1 -> 0
- net 20V: track 47.5 -> 48.0 mm
- removed copper zone on layer 1, net N$27
- removed copper zone on layer 1, net VCC
Other:
- board text added: "PWM Backlight Control"
- board text removed: "PWM Backlight"
