File: Adafruit Qualia Driver.sch (EAGLE design)
At the start: 60 parts, among them IC1 ATTINY85-20S, Q1 DMN10H170SK3-13, T1 IRLML2246, U1 LT3754, U2 MCP16321T-330E/NG, X1 0472720001, X2 FH35-51S-0.3SHW(50), X3 2.1mm

Commit message: right version
Parts:
- added R6: 20K, microbuilder:RESISTOR_0805MP
- added T2: IRLML2246, zetex:PMOSSOT23
- D1: value B260A-13-F -> PDS560-13; device microbuilder:DIODESMA -> microbuilder:DIODEPOWERDI
- Q1: value DMN10H170SK3-13 -> IRLR024NTRPBF
- SW1, SW2, SW3: value (none) -> SPST_TACT-EVQQ2; device microbuilder:SWITCH_PUSHBUTTONC&K_KSS -> adafruit:SPST_TACT-EVQQ2
- X2: value FH35-51S-0.3SHW(50) -> 502250-5191
Connections:
- removed net N$18: ON/OFF2.P, R7.1, T1.G
- new net DPP: R6.2, T2.S, X1.DP_PWR
- new net ON/OFF: ON/OFF2.P, R6.1, R7.1, T1.G, T2.G
- net 3.3V: now also T2.D; no longer X1.DP_PWR
- net BDOWN: now also SW2.S, SW2.S1; no longer SW3.P$2
- net BUP: now also SW1.S, SW1.S1; no longer SW2.P$2
- net GND: now also SW1.P, SW1.P1, SW2.P, SW2.P1, SW3.P; no longer SW1.P$1, SW2.P$1, SW3.P$1
- net MOSI: now also SW3.S; no longer SW1.P$2
Other:
- moved on the sheet: C16, LED1, ON/OFF2, R1, R7, SJ1, T1, X3
